File: V2/Circuit/Circuit.kicad_pcb (KiCad board)
At the start: 2 copper layers, 20 parts, among them J2 PinHeader-1x3, U1 TMC2209_SILENTSTEPSTICK, U2 LM338T

Commit message: Finshed all HAL and a good chunk of application layer, finalized circuit schematic
Parts:
- removed Encoder_Speed1, Encoder_Steps1: JST-5P, Connector_JST:JST_EH_B5B-EH-A_1x05_P2.50mm_Vertical
- added C3: 10nf, Resistor_THT:R_Axial_DIN0207_L6.3mm_D2.5mm_P7.62mm_Horizontal, F.Cu at (114.5, 118.0)
- added Control-mode-switch1: JST2P, Connector_JST:JST_EH_B2B-EH-A_1x02_P2.50mm_Vertical, F.Cu at (131.0, 102.7)
- added Debug1: Pin_01x03, Connector_PinHeader_2.54mm:PinHeader_1x03_P2.54mm_Vertical, F.Cu at (128.2, 131.0)
- added Encoder1: JST5P, Connector_JST:JST_EH_B5B-EH-A_1x05_P2.50mm_Vertical, F.Cu at (99.5, 84.0)
- added Encoder2: JST5P, Connector_JST:JST_EH_B5B-EH-A_1x05_P2.50mm_Vertical, F.Cu at (141.0, 91.8)
- added PowerIN1: Terminal, TerminalBlock:TerminalBlock_bornier-2_P5.08mm, F.Cu at (115.2, 59.5)
- added R5: 100, Resistor_THT:R_Axial_DIN0207_L6.3mm_D2.5mm_P7.62mm_Horizontal, F.Cu at (117.4, 125.2)
- C2: footprint Capacitor_THT:CP_Radial_D8.0mm_P3.50mm -> Capacitor_THT:CP_Radial_D5.0mm_P2.50mm
- CW-CCW-switch1, Hold-Free-switch1, Run-Button1, Stop-Button1: value JST-2P -> JST2P
- J2: value PinHeader-1x3 -> IDC-10P; footprint Connector_PinHeader_2.54mm:PinHeader_1x03_P2.54mm_Vertical -> Connector_IDC:IDC-Header_2x05_P2.54mm_Vertical
- R1: value 100 -> 220
- STC8H8K64U1: value DIP40 -> DIP28; footprint Package_DIP:DIP-40_W15.24mm_LongPads -> Package_DIP:DIP-28_W7.62mm_Socket_LongPads
- StepperOut1: value JST-4P -> JST4P
- moved R2 82.2 mm to (103.7, 60.2)
- moved R3 82.2 mm to (103.7, 64.2)
- moved StepperOut1 74.7 mm to (93.5, 101.8), turned to 90 degrees
- moved C2 67.3 mm to (126.0, 65.2)
- moved U2 58.1 mm to (118.7, 68.8)
- moved C1 57.1 mm to (96.8, 113.0), turned to 180 degrees
- moved D1 53.5 mm to (125.0, 128.5), turned to 180 degrees
- moved R1 51.4 mm to (134.4, 70.8)
- moved U1 46.0 mm to (104.7, 98.0)
- moved Run-Terminal1 44.5 mm to (144.5, 120.0), turned to 90 degrees
- moved J2 40.4 mm to (139.7, 76.0), turned to -90 degrees
- moved Stop-Button1 15.2 mm to (131.0, 113.7)
- moved CW-CCW-switch1 14.7 mm to (131.0, 97.2)
- moved Run-Button1 14.1 mm to (131.0, 119.2)
- moved Hold-Free-switch1 13.5 mm to (131.0, 108.2)
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Connections:
- CW-CCW-switch1 pad 1: GND -> CW_CCW_Switch
- CW-CCW-switch1 pad 2: CW_CCW_Switch -> GND
- D1 pad 1: Net-(D1-K) -> /TX
- Hold-Free-switch1 pad 1: GND -> HOLD_FREE_SWITCH
- Hold-Free-switch1 pad 2: HOLD_FREE_SWITCH -> GND
- J2 pad 1: Net-(J2-Pin_1) -> GND
- J2 pad 2: Net-(D1-K) -> +5V
- J2 pad 3: GND -> RW_SID
- R1 pad 1: Net-(STC8H8K64U1-Pin_22) -> Net-(J2-Pin_5)
- R1 pad 2: Net-(J2-Pin_1) -> +5V
- R2 pad 2: +24V -> +5V
- Run-Button1 pad 1: GND -> Run_Button
- Run-Button1 pad 2: Run_Button -> GND
- Run-Terminal1 pad 1: GND -> Run_Button
- Run-Terminal1 pad 2: Run_Button -> GND
- STC8H8K64U1 pad 10: unconnected-(STC8H8K64U1-Pin_10-Pad10) -> Net-(STC8H8K64U1-Pin_10)
- STC8H8K64U1 pad 11: unconnected-(STC8H8K64U1-Pin_11-Pad11) -> Encoder_DT1
- STC8H8K64U1 pad 12: unconnected-(STC8H8K64U1-Pin_12-Pad12) -> +3.3V
- STC8H8K64U1 pad 13: unconnected-(STC8H8K64U1-Pin_13-Pad13) -> GND
- STC8H8K64U1 pad 14: unconnected-(STC8H8K64U1-Pin_14-Pad14) -> GND
- STC8H8K64U1 pad 15: unconnected-(STC8H8K64U1-Pin_15-Pad15) -> Net-(D1-A)
- STC8H8K64U1 pad 16: unconnected-(STC8H8K64U1-Pin_16-Pad16) -> Net-(STC8H8K64U1-Pin_16)
- STC8H8K64U1 pad 17: unconnected-(STC8H8K64U1-Pin_17-Pad17) -> Encoder_button1
- STC8H8K64U1 pad 18: unconnected-(STC8H8K64U1-Pin_18-Pad18) -> Run_Button
- STC8H8K64U1 pad 19: unconnected-(STC8H8K64U1-Pin_19-Pad19) -> STOP_Button
- STC8H8K64U1 pad 20: GND -> HOLD_FREE_SWITCH
- STC8H8K64U1 pad 21: Net-(D1-A) -> control-mode-switch
- STC8H8K64U1 pad 22: Net-(STC8H8K64U1-Pin_22) -> CW_CCW_Switch
- STC8H8K64U1 pad 23: unconnected-(STC8H8K64U1-Pin_23-Pad23) -> Encoder_CLK2
- STC8H8K64U1 pad 24: unconnected-(STC8H8K64U1-Pin_24-Pad24) -> Encoder_DT2
- STC8H8K64U1 pad 25: unconnected-(STC8H8K64U1-Pin_25-Pad25) -> Encoder_button2
- STC8H8K64U1 pad 26: unconnected-(STC8H8K64U1-Pin_26-Pad26) -> RS_CS
- STC8H8K64U1 pad 27: unconnected-(STC8H8K64U1-Pin_27-Pad27) -> RW_SID
- STC8H8K64U1 pad 28: unconnected-(STC8H8K64U1-Pin_28-Pad28) -> E_SCLK
- STC8H8K64U1 pad 3: unconnected-(STC8H8K64U1-Pin_3-Pad3) -> Encoder_CLK1
- STC8H8K64U1 pad 4: unconnected-(STC8H8K64U1-Pin_4-Pad4) -> DIR
- STC8H8K64U1 pad 5: unconnected-(STC8H8K64U1-Pin_5-Pad5) -> STEP
- STC8H8K64U1 pad 6: unconnected-(STC8H8K64U1-Pin_6-Pad6) -> EN
- STC8H8K64U1 pad 7: unconnected-(STC8H8K64U1-Pin_7-Pad7) -> DIAG
- STC8H8K64U1 pad 8: unconnected-(STC8H8K64U1-Pin_8-Pad8) -> INDEX
- Stop-Button1 pad 1: GND -> STOP_Button
- Stop-Button1 pad 2: STOP_Button -> GND
- U1 pad 13: unconnected-(U1-SPRD-Pad13) -> GND
- U1 pad 14: unconnected-(U1-MS2-Pad14) -> GND
- U1 pad 15: unconnected-(U1-MS1-Pad15) -> GND
- U1 pad 2: unconnected-(U1-VIO-Pad2) -> +5V
- U2 pad 2: +24V -> +5V
Routing:
- net Net-(StepperOut1-Pin_4): track 0.00 -> 4.83 mm
- net Net-(StepperOut1-Pin_3): track 0.00 -> 4.82 mm
- net Net-(StepperOut1-Pin_1): track 0.00 -> 4.82 mm
- net Net-(StepperOut1-Pin_2): track 0.00 -> 4.80 mm

Commit message: almost finished pcb tracing
Parts:
- R2: value 100 -> 200
- moved R3 18.4 mm to (121.2, 70.1), turned to 180 degrees
- moved R1 14.2 mm to (132.3, 84.8)
- moved J2 12.4 mm to (127.8, 79.5), turned to 90 degrees
- moved PowerIN1 11.2 mm to (125.7, 55.6), turned to 180 degrees
- moved Encoder1 10.2 mm to (109.7, 84.3), turned to 180 degrees
- moved R2 9.96 mm to (113.5, 61.7)
- moved Encoder2 6.48 mm to (144.0, 97.5), turned to 90 degrees
- moved U2 2.81 mm to (117.3, 66.3)
- moved C2 2.38 mm to (126.0, 67.6), turned to -90 degrees
- moved C3 2.14 mm to (114.5, 120.1)
Connections:
- J2 pad 1: GND -> E_SCLK
- J2 pad 2: +5V -> GND
- J2 pad 8: E_SCLK -> +5V
- STC8H8K64U1 pad 12: +3.3V -> +5V
Routing:
- net GND: track 0.00 -> 358.8 mm
- net +5V: track 0.00 -> 163.2 mm
- net +24V: track 0.00 -> 119.9 mm
- net Encoder_button1: track 0.00 -> 63.3 mm
- net Encoder_DT1: track 0.00 -> 46.0 mm
- net Run_Button: track 0.00 -> 23.6 mm
- net Encoder_CLK2: track 0.00 -> 22.3 mm
- net Encoder_DT2: track 0.00 -> 20.9 mm
- net Encoder_button2: track 0.00 -> 20.4 mm
- net RS_CS: track 0.00 -> 19.3 mm
- net INDEX: track 0.00 -> 15.1 mm
- net RW_SID: track 0.00 -> 12.8 mm
- net Net-(STC8H8K64U1-Pin_16): track 0.00 -> 12.7 mm
- net Net-(D1-A): track 0.00 -> 12.5 mm
- net DIAG: track 0.00 -> 12.4 mm
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